Commit message: gazebo not publishing arm joint states..

File: description/robot.urdf.xacro (robot description, xacro)
@@ -1,18 +1,19 @@
 <?xml version="1.0"?>
 <robot xmlns:xacro="http://www.ros.org/wiki/xacro"  name="robot">
-    <material name="orange">
-        <color rgba="1 0.3 0.1 1"/>
-    </material>
-    <material name="blue">
-        <color rgba="0.2 0.2 1 1"/>
-    </material>
-    <material name="black">
-        <color rgba="0 0 0 1"/>
-    </material>
+	<xacro:include filename="include.xacro" />
+	<gazebo>
+        <plugin name="gazebo_ros_joint_state_publisher"
+            filename="libgazebo_joint_state_publisher.so">
+            <update_rate>20</update_rate>
+            <joint_name>stand_joint</joint_name>
+            <joint_name>arm1_joint</joint_name>
+            <joint_name>arm2_joint</joint_name>
+        </plugin>
+    </gazebo>
 	<link name="stand_link">
 		<visual>
 		    <origin xyz="0 0 0.025" rpy="0 0 0"/>
 			<geometry>
-				<box size="0.5 0.5 0.05"/>
+				<box size="0.5 0.5 0.01"/>
 			</geometry>
 			<material name="black"/>
@@ -29,4 +30,7 @@
  		 </inertial>
 	</link>
+	<gazebo reference="stand_link">
+    	<material>Gazebo/Black</material>
+	</gazebo>
     <link name="base_link">
 		<visual>
@@ -48,5 +52,8 @@
  		 </inertial>
 	</link>
-<link name="arm1_link">
+	<gazebo reference="base_link">
+    	<material>Gazebo/Orange</material>
+	</gazebo>
+	<link name="arm1_link">
 		<visual>
 			<origin xyz="0.078 0 0" rpy="0 1.57079632679 0"/>
@@ -67,5 +74,8 @@
  		 </inertial>
 	</link>
-<link name="arm2_link">
+	<gazebo reference="arm1_link">
+    	<material>Gazebo/Black</material>
+	</gazebo>
+	<link name="arm2_link">
 		<visual>
 			<origin xyz="0 0 -0.0675" rpy="0 0 0"/>
@@ -86,4 +96,7 @@
   	  </inertial>
 	</link>
+	<gazebo reference="arm2_link">
+    	<material>Gazebo/Orange</material>
+	</gazebo>
 	<joint name="stand_joint" type="fixed">
     	<parent link="stand_link"/>
