Commit message: Added anoter lauch file, fixed gazebo publisher sim

File: description/include.xacro (robot description, xacro)
@@ -17,8 +17,24 @@
             filename="libgazebo_joint_state_publisher.so">
             <update_rate>20</update_rate>
-            <joint_name>stand_joint</joint_name>
             <joint_name>arm1_joint</joint_name>
             <joint_name>arm2_joint</joint_name>
         </plugin>
     </gazebo> -->
+     <gazebo>
+        <plugin name="gazebo_ros_joint_state_publisher"
+            filename="libgazebo_ros_joint_state_publisher.so">
+            <update_rate>20</update_rate>
+            <joint_name>arm1_joint</joint_name>
+            <joint_name>arm2_joint</joint_name>
+        </plugin>
+    </gazebo>
+    <gazebo reference="base_link">
+    	<material>Gazebo/Orange</material>
+	</gazebo>
+    <gazebo reference="arm1_link">
+    	<material>Gazebo/Black</material>
+	</gazebo>
+    <gazebo reference="arm2_link">
+    	<material>Gazebo/Orange</material>
+	</gazebo>
 </robot>

File: description/robot.urdf.xacro (robot description, xacro)
@@ -1,36 +1,10 @@
 <?xml version="1.0"?>
 <robot xmlns:xacro="http://www.ros.org/wiki/xacro"  name="robot">
-	<xacro:include filename="include.xacro" />
-	<gazebo>
-        <plugin name="gazebo_ros_joint_state_publisher"
-            filename="libgazebo_joint_state_publisher.so">
-            <update_rate>20</update_rate>
-            <joint_name>stand_joint</joint_name>
-            <joint_name>arm1_joint</joint_name>
-            <joint_name>arm2_joint</joint_name>
-        </plugin>
-    </gazebo>
-	<link name="stand_link">
-		<visual>
-		    <origin xyz="0 0 0.025" rpy="0 0 0"/>
-			<geometry>
-				<box size="0.5 0.5 0.01"/>
-			</geometry>
-			<material name="black"/>
-		</visual>
-  		<collision>
-  			<origin xyz="0 0 0.1" rpy="0 0 0"/>
-			<geometry>
-				<box size="0.5 0.5 0.05"/>
-			</geometry>
-  		</collision>
-  		<inertial>
-    		<mass value="141"/>
-      		<inertia ixx="3.8" ixy="0" ixz="0" iyy="3.8" iyz="0" izz="18"/>
- 		 </inertial>
-	</link>
-	<gazebo reference="stand_link">
-    	<material>Gazebo/Black</material>
-	</gazebo>
+	 <link name="world"></link>
+	  <joint name="base_joint" type="fixed">
+        <origin xyz="1.5 1.0 0" rpy="0 0 0"/>
+        <parent link="world"/>
+        <child link="base_link"/>
+    </joint>
     <link name="base_link">
 		<visual>
@@ -52,7 +26,4 @@
  		 </inertial>
 	</link>
-	<gazebo reference="base_link">
-    	<material>Gazebo/Orange</material>
-	</gazebo>
 	<link name="arm1_link">
 		<visual>
@@ -74,7 +45,4 @@
  		 </inertial>
 	</link>
-	<gazebo reference="arm1_link">
-    	<material>Gazebo/Black</material>
-	</gazebo>
 	<link name="arm2_link">
 		<visual>
@@ -96,12 +64,4 @@
   	  </inertial>
 	</link>
-	<gazebo reference="arm2_link">
-    	<material>Gazebo/Orange</material>
-	</gazebo>
-	<joint name="stand_joint" type="fixed">
-    	<parent link="stand_link"/>
-    	<child link="base_link"/>
-    	<origin xyz="0 0 0" rpy="0 0 0"/>
-	</joint>
 	<joint name="arm1_joint" type="continuous">
     	<parent link="base_link"/>
@@ -109,4 +69,5 @@
     	<origin xyz="0 0 0.4" rpy="0 0 0"/>
   		<axis xyz = "0 0 1"/>
+		<dynamics damping="0.1"/>
 	</joint>
 	<joint name="arm2_joint" type="continuous">
@@ -115,4 +76,6 @@
     	<origin xyz="0.156 0 0" rpy="0 0 0"/>
   		<axis xyz = "1 0 0"/>
+		<dynamics damping="0.1"/>
 	</joint>
+	<xacro:include filename="include.xacro" />
 </robot>

Commit message: just in case

File: description/include.xacro (robot description, xacro)
@@ -13,12 +13,4 @@
         <color rgba="1 1 1 1"/>
     </material>
-    <!-- <gazebo>
-        <plugin name="gazebo_ros_joint_state_publisher"
-            filename="libgazebo_joint_state_publisher.so">
-            <update_rate>20</update_rate>
-            <joint_name>arm1_joint</joint_name>
-            <joint_name>arm2_joint</joint_name>
-        </plugin>
-    </gazebo> -->
      <gazebo>
         <plugin name="gazebo_ros_joint_state_publisher"
@@ -27,4 +19,5 @@
             <joint_name>arm1_joint</joint_name>
             <joint_name>arm2_joint</joint_name>
+            <joint_name>base_joint</joint_name>
         </plugin>
     </gazebo>

File: description/robot.urdf.xacro (robot description, xacro)
@@ -69,5 +69,5 @@
     	<origin xyz="0 0 0.4" rpy="0 0 0"/>
   		<axis xyz = "0 0 1"/>
-		<dynamics damping="0.1"/>
+		<dynamics damping="0.03"/>
 	</joint>
 	<joint name="arm2_joint" type="continuous">
@@ -76,5 +76,5 @@
     	<origin xyz="0.156 0 0" rpy="0 0 0"/>
   		<axis xyz = "1 0 0"/>
-		<dynamics damping="0.1"/>
+		<dynamics damping="0.02"/>
 	</joint>
 	<xacro:include filename="include.xacro" />
